File: hardware/4in1-panel.kicad_pcb (KiCad board)
At the start: 6 copper layers, 41.6 x 42.5 mm, 404 parts, among them J1 SM08B-SRSS-TB, Q1 C22385416, Q1 DOY180N03T, Q10 C22385416, Q10 DOY180N03T, Q11 C22385416, Q11 DOY180N03T, Q12 C22385416, Q12 DOY180N03T, Q13 C22385416, Q13 DOY180N03T, Q14 C22385416, Q14 DOY180N03T, Q15 C22385416, Q15 DOY180N03T, Q16 C22385416, Q16 DOY180N03T, Q17 C22385416, Q17 DOY180N03T, Q18 C22385416, Q18 DOY180N03T, Q19 C22385416, Q19 DOY180N03T, Q2 C22385416, Q2 DOY180N03T, Q20 C22385416, Q20 DOY180N03T, Q21 C22385416, Q21 DOY180N03T, Q22 C22385416, Q22 DOY180N03T, Q23 C22385416, Q23 DOY180N03T, Q24 C22385416, Q24 DOY180N03T, Q3 C22385416, Q3 DOY180N03T, Q4 C22385416, Q4 DOY180N03T, Q5 C22385416, Q5 DOY180N03T, Q6 C22385416, Q6 DOY180N03T, Q7 C22385416, Q7 DOY180N03T, Q8 C22385416, Q8 DOY180N03T, Q9 C22385416, Q9 DOY180N03T, U1 TLV76733DRVR, U10 AT32F421G8U7, U10 NSG2065Q, U11 NSG2065Q, U12 INA186A3IDCKR, U13 LMR54406DBVR, U14 FTC160808S4R7MBCA, U15 TLV76733DRVR, U2 AT32F421G8U7, U3 NSG2065Q, U4 NSG2065Q, U5 AT32F421G8U7, U5 FTC160808S4R7MBCA, U6 AT32F421G8U7, U6 NSG2065Q, U7 AT32F421G8U7, U7 NSG2065Q, U8 AT32F421G8U7, U8 NSG2065Q, U9 AT32F421G8U7, U9 NSG2065Q

Commit message: Apply DroneAid rebrand and configure upstream sync
Other:
- board text added: "DroneAid"
- board text removed: "Open"
- board text removed: "open"
